File: uino-mx250.brd (EAGLE design)
At the start: 68.6 x 53.3 mm, 32 parts, among them J1 CON_TERMINAL_BLOCK_02-5MM, U1 L4931, U2 PIC32MX250B-P

Commit message: Some minor final changes.
Parts:
- J3: value (none) -> USB_MICRO_B_2.0-TH
- moved C4 0.38 mm to (45.7, 17.4)
- moved C5 0.38 mm to (50.8, 17.4)
- moved Y1 0.38 mm to (48.3, 21.2)
Routing:
- net VCC: track 161.0 -> 166.0 mm
- net MCLR: track 126.7 -> 123.4 mm, vias 0 -> 1
- net VBUS: track 97.2 -> 97.7 mm
- net GND: vias 37 -> 39

Commit message: Added values. Added png files.
Parts:
- C1, C6: value (none) -> 4u7
- C2, C7, C8: value (none) -> 100n
- C3: value (none) -> 10u
- C4, C5: value (none) -> 27p
- D1, D2: value (none) -> SB140TA
- J3: value USB_MICRO_B_2.0-TH -> Micro USB
- R1, R2: value (none) -> 470
- R3, R4, R5, R6: value (none) -> 10k
- U1: value L4931 -> MCP1702-33
- Y1: value (none) -> 8MHz
Changed lines of the file:
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@@
 <attribute name="VALUE" x="42.926" y="53.975" size="1.27" layer="27" rot="R180"/>
 </element>
-<element name="J3" library="adi-misc" package="ZX62D-AB-5P8" value="USB_MICRO_B_2.0-TH" x="1.905" y="38.1" smashed="yes" rot="R270">
+<element name="J3" library="adi-misc" package="ZX62D-AB-5P8" value="Micro USB" x="1.905" y="38.1" smashed="yes" rot="R270">
 <attribute name="NAME" x="4.092" y="42.404" size="1.016" layer="25" ratio="18"/>
 <attribute name="VALUE" x="3.305" y="32.9" size="0.8128" layer="27" ratio="10"/>
@@
 <attribute name="VALUE" x="69.342" y="13.97" size="1.27" layer="27" font="vector" rot="R90"/>
 </element>
-<element name="U1" library="adi-misc" package="TO-92" value="L4931" x="26.67" y="16.51" smashed="yes" rot="R90">
+<element name="U1" library="adi-misc" package="TO-92" value="MCP1702-33" x="26.67" y="16.51" smashed="yes" rot="R90">
 <attribute name="NAME" x="25.273" y="19.558" size="1.016" layer="25" ratio="18"/>
 <attribute name="VALUE" x="27.94" y="19.685" size="0.4064" layer="27" ratio="10" rot="R90"/>
@@
 <attribute name="VALUE" x="12.7" y="34.69" size="0.4318" layer="27"/>
 </element>
-<element name="C7" library="rc-master" package="C025-040X018" value="" x="27.94" y="36.83" smashed="yes" rot="R180">
+<element name="C7" library="rc-master" package="C025-040X018" value="100n" x="27.94" y="36.83" smashed="yes" rot="R180">
 <attribute name="NAME" x="25.781" y="38.1" size="1.016" layer="25" ratio="18"/>
 <attribute name="VALUE" x="24.765" y="38.4175" size="0.8128" layer="27" ratio="10" rot="R180"/>
 </element>
-<element name="C1" library="rc-master" package="CTT-025-040" value="" x="20.32" y="15.24" smashed="yes" rot="R180">
+<element name="C1" library="rc-master" package="CTT-025-040" value="4u7" x="20.32" y="15.24" smashed="yes" rot="R180">
 <attribute name="NAME" x="17.399" y="16.891" size="1.016" layer="25" ratio="18"/>
 <attribute name="VALUE" x="18.415" y="17.4625" size="0.8128" layer="27" ratio="10" rot="R180"/>
 </element>
-<element name="D1" library="diode" package="DO35-7" value="" x="20.701" y="10.16" smashed="yes">
+<element name="D1" library="diode" package="DO35-7" value="SB140TA" x="20.701" y="10.16" smashed="yes">
 <attribute name="NAME" x="18.415" y="11.43" size="1.016" layer="25" ratio="18"/>
 <attribute name="VALUE" x="18.415" y="7.493" size="1.27" layer="27" ratio="10"/>
 </element>
-<element name="D2" library="diode" package="DO35-7" value="" x="20.701" y="6.35" smashed="yes">
+<element name="D2" library="diode" package="DO35-7" value="SB140TA" x="20.701" y="6.35" smashed="yes">
 <attribute name="NAME" x="18.415" y="7.62" size="1.016" layer="25" ratio="18"/>
 <attribute name="VALUE" x="18.415" y="3.683" size="1.27" layer="27" ratio="10"/>
@@
 <attribute name="VALUE" x="9.2075" y="33.655" size="0.8128" layer="27" ratio="10" rot="R180"/>
 </element>
-<element name="R2" library="rc-master" package="0207/7" value="" x="11.43" y="16.51" smashed="yes" rot="R180">
+<element name="R2" library="rc-master" package="0207/7" value="470" x="11.43" y="16.51" smashed="yes" rot="R180">
 <attribute name="NAME" x="8.255" y="17.8435" size="1.016" layer="25" ratio="18"/>
 <attribute name="VALUE" x="13.97" y="17.145" size="0.8128" layer="27" ratio="10" rot="R180"/>
 </element>
-<element name="R1" library="rc-master" package="0207/7" value="" x="11.43" y="21.59" smashed="yes" rot="R180">
+<element name="R1" library="rc-master" package="0207/7" value="470" x="11.43" y="21.59" smashed="yes" rot="R180">
 <attribute name="NAME" x="8.255" y="22.9235" size="1.016" layer="25" ratio="18"/>
 <attribute name="VALUE" x="13.97" y="22.225" size="0.8128" layer="27" ratio="10" rot="R180"/>
 </element>
-<element name="C6" library="rc-master" package="CTT-025-040" value="" x="20.32" y="20.32" smashed="yes" rot="R180">
+<element name="C6" library="rc-master" package="CTT-025-040" value="4u7" x="20.32" y="20.32" smashed="yes" rot="R180">
 <attribute name="NAME" x="17.526" y="21.971" size="1.016" layer="25" ratio="18"/>
 <attribute name="VALUE" x="18.415" y="22.5425" size="0.8128" layer="27" ratio="10" rot="R180"/>
@@
 <attribute name="VALUE" x="34.925" y="28.575" size="0.8128" layer="27" ratio="10"/>
 </element>
-<element name="R3" library="rc-master" package="0207/7" value="" x="16.51" y="27.94" smashed="yes" rot="R180">
+<element name="R3" library="rc-master" package="0207/7" value="10k" x="16.51" y="27.94" smashed="yes" rot="R180">
 <attribute name="NAME" x="13.462" y="29.2735" size="1.016" layer="25" ratio="18"/>
 <attribute name="VALUE" x="19.05" y="28.575" size="0.8128" layer="27" ratio="10" rot="R180"/>
 </element>
-<element name="R5" library="rc-master" package="0207/7" value="" x="16.51" y="45.72" smashed="yes">
+<element name="R5" library="rc-master" package="0207/7" value="10k" x="16.51" y="45.72" smashed="yes">
 <attribute name="NAME" x="13.335" y="47.0535" size="1.016" layer="25" ratio="18"/>
 <attribute name="VALUE" x="13.97" y="45.085" size="0.8128" layer="27" ratio="10"/>
 </element>
-<element name="R4" library="rc-master" package="0207/7" value="" x="16.51" y="31.75" smashed="yes" rot="R180">
+<element name="R4" library="rc-master" package="0207/7" value="10k" x="16.51" y="31.75" smashed="yes" rot="R180">
 <attribute name="NAME" x="13.462" y="33.0835" size="1.016" layer="25" ratio="18"/>
 <attribute name="VALUE" x="19.05" y="32.385" size="0.8128" layer="27" ratio="10" rot="R180"/>
 </element>
-<element name="R6" library="rc-master" package="0207/7" value="" x="16.51" y="41.91" smashed="yes">
+<element name="R6" library="rc-master" package="0207/7" value="10k" x="16.51" y="41.91" smashed="yes">
 <attribute name="NAME" x="13.335" y="43.2435" size="1.016" layer="25" ratio="18"/>
 <attribute name="VALUE" x="13.97" y="41.275" size="0.8128" layer="27" ratio="10"/>
 </element>
-<element name="C3" library="rc-master" package="C025-040X018" value="" x="48.26" y="36.83" smashed="yes" rot="R180">
+<element name="C3" library="rc-master" package="C025-040X018" value="10u" x="48.26" y="36.83" smashed="yes" rot="R180">
 <attribute name="NAME" x="46.101" y="38.1" size="1.016" layer="25" ratio="18"/>
 <attribute name="VALUE" x="45.085" y="38.4175" size="0.8128" layer="27" ratio="10" rot="R180"/>
 </element>
-<element name="Y1" library="crystal" package="HC49/S" value="" x="48.26" y="21.209" smashed="yes" rot="R180">
+<element name="Y1" library="crystal" package="HC49/S" value="8MHz" x="48.26" y="21.209" smashed="yes" rot="R180">
 <attribute name="NAME" x="42.799" y="21.59" size="1.016" layer="25" ratio="18" rot="R180"/>
 <attribute name="VALUE" x="53.34" y="25.146" size="0.8128" layer="27" ratio="10" rot="R180"/>
 </element>
-<element name="C4" library="rc-master" package="C025-040X018" value="" x="45.72" y="17.399" smashed="yes">
+<element name="C4" library="rc-master" package="C025-040X018" value="27p" x="45.72" y="17.399" smashed="yes">
 <attribute name="NAME" x="47.879" y="16.129" size="1.016" layer="25" ratio="18" rot="R180"/>
 <attribute name="VALUE" x="48.895" y="15.8115" size="0.8128" layer="27" ratio="10"/>
 </element>
-<element name="C5" library="rc-master" package="C025-040X018" value="" x="50.8" y="17.399" smashed="yes">
+<element name="C5" library="rc-master" package="C025-040X018" value="27p" x="50.8" y="17.399" smashed="yes">
 <attribute name="NAME" x="52.959" y="16.129" size="1.016" layer="25" ratio="18" rot="R180"/>
 <attribute name="VALUE" x="53.975" y="15.8115" size="0.8128" layer="27" ratio="10"/>
 </element>
-<element name="C8" library="rc-master" package="C025-040X018" value="" x="58.42" y="20.32" smashed="yes" rot="R90">
+<element name="C8" library="rc-master" package="C025-040X018" value="100n" x="58.42" y="20.32" smashed="yes" rot="R90">
 <attribute name="NAME" x="59.436" y="17.78" size="1.016" layer="25" ratio="18" rot="R180"/>
 <attribute name="VALUE" x="60.0075" y="23.495" size="0.8128" layer="27" ratio="10" rot="R90"/>
 </element>
-<element name="C2" library="rc-master" package="C025-040X018" value="" x="27.94" y="8.89" smashed="yes" rot="R90">
+<element name="C2" library="rc-master" package="C025-040X018" value="100n" x="27.94" y="8.89" smashed="yes" rot="R90">
 <attribute name="NAME" x="28.956" y="6.35" size="1.016" layer="25" ratio="18" rot="R180"/>
 <attribute name="VALUE" x="29.5275" y="12.065" size="0.8128" layer="27" ratio="10" rot="R90"/>
