File: uino-mx250.sch (EAGLE design)
At the start: 32 parts, among them J1 CON_TERMINAL_BLOCK_02-5MM, J3 USB_MICRO_B_2.0-TH, U1 L4931, U2 PIC32MX250B-P

Commit message: Some minor final changes.
Changed lines of the file:
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@@
 <part name="GND19" library="supply1" deviceset="GND" device=""/>
 <part name="GND20" library="supply1" deviceset="GND" device=""/>
-<part name="J3" library="adi-misc" deviceset="USB_MICRO_B_2.0-TH" device="" value=""/>
+<part name="J3" library="adi-misc" deviceset="USB_MICRO_B_2.0-TH" device="" value="USB_MICRO_B_2.0-TH"/>
 <part name="J2" library="SparkFun-Connectors" deviceset="M06" device="LOCK"/>
 <part name="SUPPLY1" library="SparkFun-Aesthetics" deviceset="VCC" device=""/>

Commit message: Added values. Added png files.
Parts:
- C1, C6: value (none) -> 4u7
- C2, C7, C8: value (none) -> 100n
- C3: value (none) -> 10u
- C4, C5: value (none) -> 27p
- D1, D2: value (none) -> SB140TA
- J3: value USB_MICRO_B_2.0-TH -> Micro USB
- R1, R2: value (none) -> 470
- R3, R4, R5, R6: value (none) -> 10k
- U1: value L4931 -> MCP1702-33
- Y1: value (none) -> 8MHz
Changed lines of the file:
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@@
 <layer number="91" name="Nets" color="2" fill="1" visible="yes" active="yes"/>
 <layer number="92" name="Busses" color="1" fill="1" visible="yes" active="yes"/>
-<layer number="93" name="Pins" color="2" fill="1" visible="yes" active="yes"/>
+<layer number="93" name="Pins" color="2" fill="1" visible="no" active="yes"/>
 <layer number="94" name="Symbols" color="4" fill="1" visible="yes" active="yes"/>
 <layer number="95" name="Names" color="7" fill="1" visible="yes" active="yes"/>
@@
 <part name="GND19" library="supply1" deviceset="GND" device=""/>
 <part name="GND20" library="supply1" deviceset="GND" device=""/>
-<part name="J3" library="adi-misc" deviceset="USB_MICRO_B_2.0-TH" device="" value="USB_MICRO_B_2.0-TH"/>
+<part name="J3" library="adi-misc" deviceset="USB_MICRO_B_2.0-TH" device="" value="Micro USB"/>
 <part name="J2" library="SparkFun-Connectors" deviceset="M06" device="LOCK"/>
 <part name="SUPPLY1" library="SparkFun-Aesthetics" deviceset="VCC" device=""/>
 <part name="GND2" library="supply1" deviceset="GND" device=""/>
-<part name="U1" library="adi-misc" deviceset="V_REG_MCP170X" device="" value="L4931"/>
+<part name="U1" library="adi-misc" deviceset="V_REG_MCP170X" device="" value="MCP1702-33"/>
 <part name="F1" library="adi-misc" deviceset="FUSE_PTC" device="-TH"/>
 <part name="F2" library="adi-misc" deviceset="FUSE_PTC" device="-TH"/>
-<part name="C7" library="rc-master" deviceset="C_" device="C025-040X018"/>
-<part name="C1" library="rc-master" deviceset="CP_" device="TT025-040"/>
-<part name="D1" library="diode" deviceset="SCHOTTKY-DIODE" device="DO35-7"/>
-<part name="D2" library="diode" deviceset="SCHOTTKY-DIODE" device="DO35-7"/>
+<part name="C7" library="rc-master" deviceset="C_" device="C025-040X018" value="100n"/>
+<part name="C1" library="rc-master" deviceset="CP_" device="TT025-040" value="4u7"/>
+<part name="D1" library="diode" deviceset="SCHOTTKY-DIODE" device="DO35-7" value="SB140TA"/>
+<part name="D2" library="diode" deviceset="SCHOTTKY-DIODE" device="DO35-7" value="SB140TA"/>
 <part name="LED2" library="led" deviceset="LED" device="3MM" value="Green"/>
 <part name="LED1" library="led" deviceset="LED" device="3MM" value="Blue"/>
 <part name="S2" library="adi-misc" deviceset="TL1100X" device="" value=""/>
 <part name="S1" library="adi-misc" deviceset="TL1100X" device="" value=""/>
-<part name="R2" library="rc-master" deviceset="R_" device="X0207/7"/>
-<part name="R1" library="rc-master" deviceset="R_" device="X0207/7"/>
-<part name="C6" library="rc-master" deviceset="CP_" device="TT025-040"/>
+<part name="R2" library="rc-master" deviceset="R_" device="X0207/7" value="470"/>
+<part name="R1" library="rc-master" deviceset="R_" device="X0207/7" value="470"/>
+<part name="C6" library="rc-master" deviceset="CP_" device="TT025-040" value="4u7"/>
 <part name="GND13" library="supply1" deviceset="GND" device=""/>
 <part name="GND12" library="supply1" deviceset="GND" device=""/>
@@
 <part name="U2" library="adi-pic" deviceset="PIC32MX250B" device="-P"/>
 <part name="SUPPLY4" library="SparkFun-Aesthetics" deviceset="VCC" device=""/>
-<part name="R3" library="rc-master" deviceset="R_" device="X0207/7"/>
-<part name="R5" library="rc-master" deviceset="R_" device="X0207/7"/>
-<part name="R4" library="rc-master" deviceset="R_" device="X0207/7"/>
-<part name="R6" library="rc-master" deviceset="R_" device="X0207/7"/>
+<part name="R3" library="rc-master" deviceset="R_" device="X0207/7" value="10k"/>
+<part name="R5" library="rc-master" deviceset="R_" device="X0207/7" value="10k"/>
+<part name="R4" library="rc-master" deviceset="R_" device="X0207/7" value="10k"/>
+<part name="R6" library="rc-master" deviceset="R_" device="X0207/7" value="10k"/>
 <part name="GND17" library="supply1" deviceset="GND" device=""/>
 <part name="GND18" library="supply1" deviceset="GND" device=""/>
@@
 <part name="SUPPLY2" library="SparkFun-Aesthetics" deviceset="VCC" device=""/>
 <part name="GND11" library="supply1" deviceset="GND" device=""/>
-<part name="C3" library="rc-master" deviceset="C_" device="C025-040X018"/>
+<part name="C3" library="rc-master" deviceset="C_" device="C025-040X018" value="10u"/>
 <part name="GND10" library="supply1" deviceset="GND" device=""/>
 <part name="GND3" library="supply1" deviceset="GND" device=""/>
-<part name="Y1" library="crystal" deviceset="CRYTAL" device="HC49S"/>
-<part name="C4" library="rc-master" deviceset="C_" device="C025-040X018"/>
-<part name="C5" library="rc-master" deviceset="C_" device="C025-040X018"/>
+<part name="Y1" library="crystal" deviceset="CRYTAL" device="HC49S" value="8MHz"/>
+<part name="C4" library="rc-master" deviceset="C_" device="C025-040X018" value="27p"/>
+<part name="C5" library="rc-master" deviceset="C_" device="C025-040X018" value="27p"/>
 <part name="GND8" library="supply1" deviceset="GND" device=""/>
 <part name="GND7" library="supply1" deviceset="GND" device=""/>
 <part name="SUPPLY5" library="SparkFun-Aesthetics" deviceset="VCC" device=""/>
-<part name="C8" library="rc-master" deviceset="C_" device="C025-040X018"/>
+<part name="C8" library="rc-master" deviceset="C_" device="C025-040X018" value="100n"/>
 <part name="GND14" library="supply1" deviceset="GND" device=""/>
-<part name="C2" library="rc-master" deviceset="C_" device="C025-040X018"/>
+<part name="C2" library="rc-master" deviceset="C_" device="C025-040X018" value="100n"/>
 <part name="GND6" library="supply1" deviceset="GND" device=""/>
 </parts>
@@
 <instance part="GND19" gate="1" x="187.96" y="127"/>
 <instance part="GND20" gate="1" x="187.96" y="48.26"/>
-<instance part="J3" gate="G$1" x="2.54" y="83.82" rot="MR0"/>
+<instance part="J3" gate="G$1" x="2.54" y="83.82" smashed="yes" rot="MR0">
+<attribute name="NAME" x="7.62" y="95.25" size="1.778" layer="95" rot="MR0"/>
+<attribute name="VALUE" x="7.62" y="92.456" size="1.778" layer="96" rot="MR0"/>
+</instance>
 <instance part="J2" gate="G$1" x="0" y="116.84" rot="MR180"/>
 <instance part="SUPPLY1" gate="G$1" x="7.62" y="124.46" rot="MR0"/>
 <instance part="GND2" gate="1" x="7.62" y="104.14" rot="MR0"/>
-<instance part="U1" gate="G$1" x="43.18" y="160.02"/>
+<instance part="U1" gate="G$1" x="43.18" y="160.02" smashed="yes">
+<attribute name="NAME" x="45.72" y="152.4" size="1.778" layer="95"/>
+<attribute name="VALUE" x="36.322" y="164.338" size="1.778" layer="96"/>
+</instance>
 <instance part="F1" gate="G$1" x="12.7" y="157.48"/>
 <instance part="F2" gate="G$1" x="20.32" y="86.36"/>
 <instance part="C7" gate="G$1" x="68.58" y="152.4" rot="R90"/>
 <instance part="C1" gate="G$1" x="30.48" y="152.4" rot="R90"/>
-<instance part="D1" gate="G$1" x="22.86" y="170.18"/>
-<instance part="D2" gate="G$1" x="22.86" y="152.4" rot="R90"/>
+<instance part="D1" gate="G$1" x="22.86" y="170.18" smashed="yes">
+<attribute name="NAME" x="20.955" y="172.085" size="1.778" layer="95"/>
+<attribute name="VALUE" x="17.145" y="166.37" size="1.778" layer="96"/>
+</instance>
+<instance part="D2" gate="G$1" x="22.86" y="152.4" smashed="yes" rot="R90">
+<attribute name="NAME" x="20.955" y="150.495" size="1.778" layer="95" rot="R90"/>
+<attribute name="VALUE" x="26.67" y="146.685" size="1.778" layer="96" rot="R90"/>
+</instance>
 <instance part="LED2" gate="G$1" x="111.76" y="167.64"/>
 <instance part="LED1" gate="G$1" x="96.52" y="167.64"/>
@@
 <instance part="GND10" gate="1" x="43.18" y="50.8"/>
 <instance part="GND3" gate="1" x="12.7" y="66.04"/>
-<instance part="Y1" gate="G$1" x="53.34" y="99.06" rot="R90"/>
+<instance part="Y1" gate="G$1" x="53.34" y="99.06" smashed="yes" rot="R90">
+<attribute name="NAME" x="51.054" y="97.79" size="1.778" layer="95" rot="R90"/>
+<attribute name="VALUE" x="57.658" y="96.52" size="1.778" layer="96" rot="R90"/>
+</instance>
 <instance part="C4" gate="G$1" x="45.72" y="104.14"/>
 <instance part="C5" gate="G$1" x="45.72" y="93.98"/>
